File: pcb_desings/radar_d1_mini_pcb/radar_d1_mini_pcb.kicad_pcb (KiCad board)
At the start: 2 copper layers, 81.3 x 28.7 mm, 8 parts

Commit message: Added gerbers radar pcb v0.0.1 adding 3mm hole
Other:
- outline, holes or cut-outs redrawn
- board text added: "v0.0.1"
- board text removed: "v0.0"
Changed lines of the file:
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@@
   (general
     (thickness 1.6)
-    (drawings 37)
+    (drawings 40)
     (tracks 93)
     (zones 0)
@@
       (padsonsilk false)
       (subtractmaskfromsilk false)
-      (outputformat 4)
+      (outputformat 1)
       (mirror false)
       (drillshape 0)
       (scaleselection 1)
-      (outputdirectory "gerber/pdf/"))
+      (outputdirectory "gerber/"))
   )
   (net 0 "")
@@
     )
   )
-  (gr_text v0.0 (at 163.83 122.428) (layer F.SilkS)
+  (gr_circle (center 114.046 127.762) (end 115.646 127.762) (layer Edge.Cuts) (width 0.15))
+  (dimension 16.51 (width 0.3) (layer Dwgs.User)
+    (gr_text "16.510 mm" (at 105.791 135.704) (layer Dwgs.User)
+      (effects (font (size 1.5 1.5) (thickness 0.3)))
+    )
+    (feature1 (pts (xy 114.046 127.762) (xy 114.046 134.190421)))
+    (feature2 (pts (xy 97.536 127.762) (xy 97.536 134.190421)))
+    (crossbar (pts (xy 97.536 133.604) (xy 114.046 133.604)))
+    (arrow1a (pts (xy 114.046 133.604) (xy 112.919496 134.190421)))
+    (arrow1b (pts (xy 114.046 133.604) (xy 112.919496 133.017579)))
+    (arrow2a (pts (xy 97.536 133.604) (xy 98.662504 134.190421)))
+    (arrow2b (pts (xy 97.536 133.604) (xy 98.662504 133.017579)))
+  )
+  (dimension 16.002 (width 0.3) (layer Dwgs.User)
+    (gr_text "16.002 mm" (at 90.102 135.763 90) (layer Dwgs.User)
+      (effects (font (size 1.5 1.5) (thickness 0.3)))
+    )
+    (feature1 (pts (xy 97.536 127.762) (xy 91.615579 127.762)))
+    (feature2 (pts (xy 97.536 143.764) (xy 91.615579 143.764)))
+    (crossbar (pts (xy 92.202 143.764) (xy 92.202 127.762)))
+    (arrow1a (pts (xy 92.202 127.762) (xy 92.788421 128.888504)))
+    (arrow1b (pts (xy 92.202 127.762) (xy 91.615579 128.888504)))
+    (arrow2a (pts (xy 92.202 143.764) (xy 92.788421 142.637496)))
+    (arrow2b (pts (xy 92.202 143.764) (xy 91.615579 142.637496)))
+  )
+  (gr_text v0.0.1 (at 163.576 122.428) (layer F.SilkS)
     (effects (font (size 1 1) (thickness 0.25)))
   )
-  (gr_text Optimun_radar (at 157.48 120.142) (layer F.SilkS)
+  (gr_text Optimun_radar (at 157.734 120.142) (layer F.SilkS)
     (effects (font (size 1.5 1.5) (thickness 0.375)))
   )

Commit message: Updated pcb label name
Other:
- board text added: "Optimum_ODS"
- board text removed: "Optimun_radar"
Changed lines of the file:
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@@
       (padsonsilk false)
       (subtractmaskfromsilk false)
-      (outputformat 1)
+      (outputformat 4)
       (mirror false)
       (drillshape 0)
       (scaleselection 1)
-      (outputdirectory "gerber/"))
+      (outputdirectory "gerber-pdf/"))
   )
   (net 0 "")
@@
     (effects (font (size 1 1) (thickness 0.25)))
   )
-  (gr_text Optimun_radar (at 157.734 120.142) (layer F.SilkS)
+  (gr_text Optimum_ODS (at 157.734 120.142) (layer F.SilkS)
     (effects (font (size 1.5 1.5) (thickness 0.375)))
   )
